File: Circuits/Eagle/projet_electronique1.brd (EAGLE design)
At the start: 100 x 80 mm, 13 parts, among them IC1 74LS48N, IC2 74LS48N, IC3 LM35CZ

Commit message: Final commit
Parts:
- removed D2: HLMP6, display-hp:HLMP6
- removed D3: (no value), special:7SEG-13
- removed IC2: 74LS48N, 74xx-eu:DIL16
- removed IC3: LM35CZ, lm35:TO92
- removed R8, R9: (no value), rcl:0204/7
- removed SV2: (no value), con-lstb:MA08-1
- added CX1, CX2, CX3, CX4: 1u, rcl:XC10B5
- added CX5, CX6: 15p, rcl:XC10B5
- added CX7: 680n, rcl:XC10B5
- added S1: (no value), switch-omron:B3F-10XX
- added SV5: (no value), con-lstb:MA08-1
- added U1: PIC16F877P, pic16f87x:DIL40
- added X3: (no value), con-subd:F09V
- D1: value (none) -> HLMP6; device special:7SEG-13 -> display-hp:HLMP6
- IC1: value 74LS48N -> MAX232; device 74xx-eu:DIL16 -> maxim:DIL16
- moved SV3 91.4 mm to (87.6, 3.81), turned to 180 degrees
- moved SV4 71.1 mm to (53.3, 68.6)
- moved D1 66.5 mm to (14.0, 73.7)
- moved IC1 54.0 mm to (64.8, 68.6), turned to 90 degrees
- moved X1 32.2 mm to (8.89, 36.8), turned to 0 degrees
- moved SV1 12.0 mm to (20.3, 61.0)
Connections:
- removed net N$3: IC2.1, SV1.4
- new net N$25: SV1.3, U1.6
- new net N$30: SV3.6, U1.21
- new net N$31: SV3.5, U1.22
- new net N$32: SV3.4, U1.27
- new net N$33: SV3.3, U1.28
- new net N$36: SV4.5, U1.37
- new net N$37: SV4.6, U1.38
- new net N$38: SV4.7, U1.39
- new net N$39: SV4.8, U1.40
- new net N$40: SV5.8, U1.9
- new net N$41: SV5.7, U1.10
- new net N$42: SV5.6, U1.15
- new net N$43: SV5.5, U1.16
- new net N$44: SV5.4, U1.17
- new net N$45: SV5.3, U1.18
- new net N$46: SV5.2, U1.23
- new net N$47: SV5.1, U1.24
- new net S$1: D1.K
- new net S$3: D1.A
- net GND: now also CX4.2, CX5.2, CX6.2, IC1.10, IC1.15, X3.7, X3.8; no longer IC1.8, IC2.8
- net N$1: now also X1.1; no longer IC3.2, SV1.7
- net N$10: now also CX2.2, IC1.5; no longer D1.2, IC2.10
- net N$11: now also CX3.1, IC1.2; no longer D1.1, IC2.9
- net N$12: now also CX4.1, IC1.6; no longer D1.9, IC2.15
- net N$13: now also IC1.11, U1.25; no longer D1.10, IC2.14
- net N$14: now also IC1.12, U1.26; no longer IC1.7, SV2.8
- net N$15: now also SV1.7, U1.2; no longer IC1.1, SV2.7
- net N$16: now also IC1.14, X3.3; no longer IC1.2, SV2.6
- net N$17: now also IC1.13, X3.2; no longer IC1.6, SV2.5
- net N$18: now also SV4.1, U1.33; no longer IC1.3, IC1.4, SV2.4
- net N$19: now also SV4.2, U1.34; no longer D3.7, IC1.13
- net N$2: now also CX7.1, S1.2; no longer IC2.7, SV1.5
- net N$20: now also SV4.3, U1.35; no longer D3.6, IC1.12
- net N$21: now also SV4.4, U1.36; no longer D3.4, IC1.11
- net N$22: now also SV1.6, U1.3; no longer D3.2, IC1.10
- net N$23: now also SV1.5, U1.4; no longer D3.1, IC1.9
- net N$24: now also SV1.4, U1.5; no longer D3.9, IC1.15
- net N$26: now also SV1.2, U1.7; no longer IC3.1, X1.1
- net N$27: now also SV1.1, U1.8; no longer D3.10, IC1.14
- net N$28: now also SV3.8, U1.19; no longer D2.A, SV2.2
- net N$29: now also SV3.7, U1.20; no longer IC3.3, R8.2, R9.2, X1.2
- net N$34: now also SV3.2, U1.29; no longer D1.8, R9.1
- net N$35: now also SV3.1, U1.30; no longer D2.K, D3.8, R8.1
- net N$4: now also CX5.1, U1.13; no longer SV1.3
- net N$5: now also CX1.1, IC1.1; no longer IC2.6, SV1.2
- net N$6: now also CX7.2, S1.4, X1.2; no longer IC2.3, IC2.4, SV1.1
- net N$7: now also CX6.1, U1.14; no longer D1.7, IC2.13
- net N$8: now also CX1.2, IC1.3; no longer D1.6, IC2.12
- net N$9: now also CX2.1, IC1.4; no longer D1.4, IC2.11
- net VCC: now also CX3.2; no longer IC2.16
Routing:
- net N$1: track 166.5 -> 0.00 mm
- net GND: track 30.6 -> 149.8 mm
- net N$34: track 19.4 -> 126.2 mm
- net N$33: track 0.00 -> 102.3 mm
- net N$30: track 0.00 -> 93.9 mm
- net N$31: track 0.00 -> 93.4 mm
- net N$12: track 59.1 -> 150.4 mm
- net N$46: track 0.00 -> 71.7 mm
- net N$25: track 78.0 -> 7.62 mm
- net N$19: track 80.6 -> 12.8 mm
- net N$8: track 82.5 -> 15.3 mm
- net S$3: track 0.00 -> 64.8 mm
- net N$35: track 155.5 -> 93.0 mm
- net N$21: track 74.3 -> 12.8 mm
- net N$24: track 68.9 -> 7.62 mm
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- added copper zone on layer 16, net N$48
- removed copper zone on layer 16, net N$30
Other:
- board text removed: "Grenier Maxime Moers Tristan Omuruon M. Francis Willame Arnaud 2TL2"
