File: Circuits/Eagle/Plaque 1/projet_electronique.brd (EAGLE design)
At the start: 100 x 80 mm, 16 parts, among them IC1 MAX232, U1 PIC16F877P

Commit message: Final commit
Parts:
- removed Q1: (no value), special:Q
- removed SV2: (no value), con-lstb:MA07-1
- added SV3, SV4, SV5: (no value), con-lstb:MA08-1
- moved S1 89.1 mm to (67.3, 73.7)
- moved CX6 85.2 mm to (5.08, 8.89), turned to 270 degrees
- moved X3 74.6 mm to (90.2, 62.2), turned to 90 degrees
- moved SV1 66.7 mm to (24.1, 48.3), turned to 90 degrees
- moved X1 52.1 mm to (14.0, 73.7)
- moved CX5 49.5 mm to (11.4, 55.9), turned to 90 degrees
- moved CX4 46.6 mm to (45.7, 66.0), turned to 180 degrees
- moved CX3 43.2 mm to (67.3, 64.8), turned to 180 degrees
- moved CX2 20.5 mm to (95.2, 31.8), turned to 90 degrees
- moved CX1 19.1 mm to (95.2, 8.89)
- moved D1 11.5 mm to (6.35, 39.4)
- moved U1 10.9 mm to (47.0, 34.3), turned to 270 degrees
- moved CX7 5.39 mm to (6.35, 25.4), turned to 90 degrees
- moved IC1 5.08 mm to (85.1, 19.1), turned to 90 degrees
Connections:
- net LM35 renamed N$15
- removed net ALERTLED: SV2.7, U1.15
- removed net DECODER1: SV2.1, U1.33
- removed net DECODER2: SV1.5, U1.19
- removed net N$2: CX7.1, D1.A, S1.2
- new net N$26: SV1.2, U1.7
- new net N$27: SV1.1, U1.8
- new net N$28: SV3.8, U1.19
- new net N$29: SV3.7, U1.20
- new net N$30: SV3.6, U1.21
- new net N$31: SV3.5, U1.22
- new net N$32: SV3.4, U1.27
- new net N$33: SV3.3, U1.28
- new net N$34: SV3.2, U1.29
- new net N$35: SV3.1, U1.30
- new net N$36: SV4.5, U1.37
- new net N$37: SV4.6, U1.38
- new net N$38: SV4.7, U1.39
- new net N$39: SV4.8, U1.40
- new net N$40: SV5.8, U1.9
- new net N$41: SV5.7, U1.10
- new net N$42: SV5.6, U1.15
- new net N$43: SV5.5, U1.16
- new net N$44: SV5.4, U1.17
- new net N$45: SV5.3, U1.18
- new net N$46: SV5.2, U1.23
- new net N$47: SV5.1, U1.24
- net GND: no longer CX4.2, CX5.2, CX6.2, IC1.10, X3.7, X3.8
- net N$1: now also D1.A; no longer X1.1
- net N$18: now also SV4.1, U1.33; no longer SV2.2, U1.34
- net N$19: now also SV4.2, U1.34; no longer SV2.3, U1.35
- net N$20: now also SV4.3, U1.35; no longer SV2.4, U1.36
- net N$21: now also SV4.4, U1.36; no longer SV2.5, U1.37
- net N$22: now also SV1.6, U1.3; no longer SV1.4, U1.20
- net N$23: now also SV1.5, U1.4; no longer SV1.3, U1.21
- net N$24: now also SV1.4, U1.5; no longer SV1.2, U1.22
- net N$25: now also SV1.3, U1.6; no longer SV1.1, U1.27
- net N$3: now also CX4.2, CX5.2, CX6.2, CX7.2, IC1.10, S1.4, X1.2, X3.5, X3.7, X3.8; no longer U1.1
- net N$6: now also CX3.2, CX7.1, S1.2, U1.1, X1.1; no longer CX7.2, S1.4, X1.2
- net VCC: no longer CX3.2
Routing:
- net N$3: track 30.2 -> 294.1 mm
- net N$11: track 13.0 -> 238.0 mm
- net N$6: track 30.6 -> 250.8 mm
- net N$22: track 153.9 -> 15.2 mm
- net N$14: track 31.9 -> 150.8 mm
- net N$41: track 0.00 -> 110.7 mm
- net N$7: track 147.2 -> 39.0 mm
- net GND: track 102.2 -> 0.00 mm
- net ALERTLED: track 72.7 -> 0.00 mm
- net N$15: track 86.7 -> 15.2 mm
- net N$12: track 32.4 -> 98.8 mm
- net DECODER2: track 64.4 -> 0.00 mm
- net N$46: track 0.00 -> 57.1 mm
- net N$4: track 16.1 -> 66.0 mm
- net N$47: track 0.00 -> 46.9 mm
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- added copper zone on layer 16, net N$50
