File: Circuits/Eagle/Plaque 2/plaque2.sch (EAGLE design)
At the start: 9 parts, among them IC1 74LS48N, IC2 74LS48N, IC3 LM35CZ

Commit message: Final commit
Parts:
- removed JP4: (no value), pinhead:PINHD-1X2
- removed LED1: (no value), eagle-ltspice:LED_E
- added D2: HLMP6, display-hp:HLMP6
- added R8, R9: (no value), rcl:R-EU_0204/7
- added SV3, SV4: (no value), con-lstb:MA08-1
- added X1: (no value), con-ptr500:AK500/2-H
- SV2: device con-lstb:MA07-1 -> con-lstb:MA08-1
Connections:
- removed net GND: D1.CK2, D3.CK2, IC3.GND, LED1.C
- removed net N$25: D3.A
- removed net N$30: D3.D
- removed net N$31: D3.E
- removed net N$32: D3.F
- removed net N$33: D3.G
- removed net N$36: D1.C
- removed net N$37: D1.D
- removed net N$38: D1.E
- removed net N$39: D1.F
- removed net N$40: D1.G
- removed net VCC: IC3.+VS
- net N$10: now also D1.D
- net N$11: now also D1.E
- net N$12: now also D1.F
- net N$13: now also D1.G
- net N$14: now also SV2.8; no longer SV2.7
- net N$15: now also SV2.7; no longer SV2.6
- net N$16: now also SV2.6; no longer SV2.5
- net N$17: now also SV2.5; no longer SV2.4
- net N$18: now also SV2.4; no longer SV2.3
- net N$19: now also D3.A
- net N$20: now also D3.B
- net N$21: now also D3.C
- net N$22: now also D3.D
- net N$23: now also D3.E
- net N$24: now also D3.F
- net N$26: now also IC3.+VS, X1-1.KL; no longer D3.B
- net N$27: now also D3.G
- net N$28: now also D2.A, SV2.2; no longer LED1.A, SV2.1
- net N$29: now also IC3.GND, R8.2, R9.2, X1-2.KL; no longer D3.C
- net N$34: now also D1.CK2, R9.1; no longer D1.A
- net N$35: now also D2.K, D3.CK2, R8.1; no longer D1.B
- net N$7: now also D1.A
- net N$8: now also D1.B
- net N$9: now also D1.C
